File: stepDown.sch (KiCad schematic (older format))
At the start: 48 parts, among them P1 ScrewIN, P2 PowerPoleOUT, P3 PowerPoleIN, P4 ScrewOUT, Q1 M1, Q2 M2, Q3 M3, Q4 M4, U1 LM25119

Commit message: weiter gemacht...
Parts:
- removed D3: LED, LEDs:LED-3MM, symbol LED
- added C20: Cout, Capacitors_SMD:C_1210, symbol C
- added C21, C22: 300p, Capacitors_SMD:C_0402, symbol C
- added C23: Cinx, Capacitors_SMD:C_0805, symbol C
- added R13, R14, R15: 4,7, Resistors_SMD:R_0603, symbol R
- added R16, R17, R18, R19: 10, Resistors_SMD:R_0603, symbol R
- R11: value Rled1 -> 4,7
Connections:
- net +12V: now also C20.1
- net +24V: now also P1.1 (P1), C23.1; no longer R11.1
- net CS1: now also C21.2, R16.2; no longer Q2.S, R7.1
- net CS2: now also C22.2, R18.2; no longer Q4.S, R10.1
- net CSG1: now also C21.1, R17.1; no longer NT1.1
- net CSG2: now also C22.1, R19.2; no longer NT2.1
- net GND: now also C20.2, C23.2; no longer P1.1 (P1)
- net HO1: now also R11.2; no longer Q1.G
- net HO2: now also R14.2; no longer Q3.G
- net LO1: now also R13.2; no longer Q2.G
- net LO2: now also R15.2; no longer Q4.G
- new net: Q1.G, R11.1
- new net: Q2.G, R13.1
- new net: Q2.S, R16.1, R7.1
- new net: Q3.G, R14.1
- new net: Q4.G, R15.1
- new net: Q4.S, R10.1, R18.1
- new net: NT1.1, R17.2
- new net: NT2.1, R19.1
Other:
- moved on the sheet: NT2, R10
